File: alturia-magswitch.sch (KiCad schematic (older format))
At the start: 20 parts, among them J101 Conn_01x01, J102 Conn_01x01, J103 Conn_01x01, J104 Conn_01x01, Q101 SISS27ADN-T1-GE3, Q102 Q_NMOS_GSD, U101 DRV5032FB, U102 AP7383-33WR-7, U103 ATtiny4-TS

Commit message: fix wrongly connected power mosfet
Signed-off-by: Thomas Schmid <tom@binary-kitchen.de>
Parts:
- R102: value 1k -> 10k
Connections:
- net OUT: now also J101.1 (Pin_1), Q101.5 (D); no longer J102.1 (Pin_1), Q101.1 (S), Q101.2 (S), Q101.3 (S)
- net VPP: now also J102.1 (Pin_1), Q101.1 (S), Q101.2 (S), Q101.3 (S); no longer J101.1 (Pin_1), Q101.5 (D)
Other:
- moved on the sheet: J101, J102
Changed lines of the file:
@@
 P 9700 2700
 F 0 "R102" H 9770 2746 50  0000 L CNN
-F 1 "1k" H 9770 2655 50  0000 L CNN
+F 1 "10k" H 9770 2655 50  0000 L CNN
 F 2 "Resistor_SMD:R_0402_1005Metric" V 9630 2700 50  0001 C CNN
 F 3 "~" H 9700 2700 50  0001 C CNN
@@
 L Connector_Generic:Conn_01x01 J101
 U 1 1 5EDDE63C
+P 8600 1300
+F 0 "J101" H 8680 1342 50  0000 L CNN
+F 1 "Conn_01x01" H 8680 1251 50  0000 L CNN
+F 2 "Connector_Wire:SolderWire-1.5sqmm_1x01_D1.7mm_OD3.9mm" H 8600 1300 50  0001 C CNN
+F 3 "~" H 8600 1300 50  0001 C CNN
+	1    8600 1300
+	1    0    0    -1
+$EndComp
+$Comp
+L Connector_Generic:Conn_01x01 J102
+U 1 1 5EDDE98D
 P 8600 1100
-F 0 "J101" H 8680 1142 50  0000 L CNN
+F 0 "J102" H 8680 1142 50  0000 L CNN
 F 1 "Conn_01x01" H 8680 1051 50  0000 L CNN
 F 2 "Connector_Wire:SolderWire-1.5sqmm_1x01_D1.7mm_OD3.9mm" H 8600 1100 50  0001 C CNN
 F 3 "~" H 8600 1100 50  0001 C CNN
 	1    8600 1100
-	1    0    0    -1
-$EndComp
-$Comp
-L Connector_Generic:Conn_01x01 J102
-U 1 1 5EDDE98D
-P 8600 1300
-F 0 "J102" H 8680 1342 50  0000 L CNN
-F 1 "Conn_01x01" H 8680 1251 50  0000 L CNN
-F 2 "Connector_Wire:SolderWire-1.5sqmm_1x01_D1.7mm_OD3.9mm" H 8600 1300 50  0001 C CNN
-F 3 "~" H 8600 1300 50  0001 C CNN
-	1    8600 1300
 	1    0    0    -1
 $EndComp
@@
 F 4 "SI7149ADP" H 10100 3000 50  0001 C CNN "Partnumber"
 	1    10100 3000
-	1    0    0    -1
-$EndComp
-Wire Wire Line
+	1    0    0    1
+$EndComp
+Wire Wire Line
